Commit message: Map 생성 및 기타 버그 수정

File: src/dqn_autonomous/urdf/robot.urdf (robot description, URDF)
Before this commit: robot dqn_4wheel_car, 11 links, 10 joints
Links:
- removed link front_left_wheel_stripe
- removed link front_right_wheel_stripe
- removed link rear_left_wheel_stripe
- removed link rear_right_wheel_stripe
- added link front_left_wheel_stripe_1; visual box size=0.11 0.01 0.001
- added link front_left_wheel_stripe_2; visual box size=0.11 0.01 0.001
- added link front_right_wheel_stripe_1; visual box size=0.11 0.01 0.001
- added link front_right_wheel_stripe_2; visual box size=0.11 0.01 0.001
- added link rear_left_wheel_stripe_1; visual box size=0.11 0.01 0.001
- added link rear_left_wheel_stripe_2; visual box size=0.11 0.01 0.001
- added link rear_right_wheel_stripe_1; visual box size=0.11 0.01 0.001
- added link rear_right_wheel_stripe_2; visual box size=0.11 0.01 0.001
Joints:
- removed joint front_left_wheel_stripe_joint
- removed joint front_right_wheel_stripe_joint
- removed joint rear_left_wheel_stripe_joint
- removed joint rear_right_wheel_stripe_joint
- added joint front_left_wheel_stripe_1_joint: type fixed, parent front_left_wheel, child front_left_wheel_stripe_1, origin xyz=0 0 0.021 rpy=0 0 0
- added joint front_left_wheel_stripe_2_joint: type fixed, parent front_left_wheel, child front_left_wheel_stripe_2, origin xyz=0 0 -0.021 rpy=0 0 0
- added joint front_right_wheel_stripe_1_joint: type fixed, parent front_right_wheel, child front_right_wheel_stripe_1, origin xyz=0 0 0.021 rpy=0 0 0
- added joint front_right_wheel_stripe_2_joint: type fixed, parent front_right_wheel, child front_right_wheel_stripe_2, origin xyz=0 0 -0.021 rpy=0 0 0
- added joint rear_left_wheel_stripe_1_joint: type fixed, parent rear_left_wheel, child rear_left_wheel_stripe_1, origin xyz=0 0 0.021 rpy=0 0 0
- added joint rear_left_wheel_stripe_2_joint: type fixed, parent rear_left_wheel, child rear_left_wheel_stripe_2, origin xyz=0 0 -0.021 rpy=0 0 0
- added joint rear_right_wheel_stripe_1_joint: type fixed, parent rear_right_wheel, child rear_right_wheel_stripe_1, origin xyz=0 0 0.021 rpy=0 0 0
- added joint rear_right_wheel_stripe_2_joint: type fixed, parent rear_right_wheel, child rear_right_wheel_stripe_2, origin xyz=0 0 -0.021 rpy=0 0 0

Commit message: 전체적인 기반 마련

File: src/dqn_autonomous/urdf/robot.urdf (robot description, URDF)
Before this commit: robot dqn_4wheel_car, 15 links, 14 joints
Links:
- removed link front_left_wheel_stripe_1
- removed link front_left_wheel_stripe_2
- removed link front_right_wheel_stripe_1
- removed link front_right_wheel_stripe_2
- removed link rear_left_wheel_stripe_1
- removed link rear_left_wheel_stripe_2
- removed link rear_right_wheel_stripe_1
- removed link rear_right_wheel_stripe_2
- link base_link: geometry visual mesh filename=package://dqn_autonomous/urdf/meshes/vehicle.obj scale=0.75 0.75 0.75
- link front_left_wheel: geometry visual mesh filename=package://dqn_autonomous/urdf/meshes/wheel.obj scale=0.75 0.75 0.75
- link front_right_wheel: geometry visual mesh filename=package://dqn_autonomous/urdf/meshes/wheel.obj scale=0.75 0.75 0.75
- link lidar_link: geometry visual cylinder length=0.0375 radius=0.03
- link rear_left_wheel: geometry visual mesh filename=package://dqn_autonomous/urdf/meshes/wheel.obj scale=0.75 0.75 0.75
- link rear_right_wheel: geometry visual mesh filename=package://dqn_autonomous/urdf/meshes/wheel.obj scale=0.75 0.75 0.75
Joints:
- removed joint front_left_wheel_stripe_1_joint
- removed joint front_left_wheel_stripe_2_joint
- removed joint front_right_wheel_stripe_1_joint
- removed joint front_right_wheel_stripe_2_joint
- removed joint rear_left_wheel_stripe_1_joint
- removed joint rear_left_wheel_stripe_2_joint
- removed joint rear_right_wheel_stripe_1_joint
- removed joint rear_right_wheel_stripe_2_joint
- joint base_joint: origin xyz=0 0 0.08 rpy=0 0 0 -> xyz=0 0 0.165 rpy=0 0 0
- joint front_left_wheel_joint: origin xyz=0.15 0.12 -0.02 rpy=-1.5708 0 0 -> xyz=0.1725 0.135 -0.105 rpy=-1.5708 0 0
- joint front_right_wheel_joint: origin xyz=0.15 -0.12 -0.02 rpy=-1.5708 0 0 -> xyz=0.1725 -0.135 -0.105 rpy=-1.5708 0 0
- joint lidar_joint: origin xyz=0.0 0.0 0.075 rpy=0 0 0 -> xyz=0.0 0.0 0.05625 rpy=0 0 0
- joint rear_left_wheel_joint: origin xyz=-0.15 0.12 -0.02 rpy=-1.5708 0 0 -> xyz=-0.24 0.135 -0.105 rpy=-1.5708 0 0
- joint rear_right_wheel_joint: origin xyz=-0.15 -0.12 -0.02 rpy=-1.5708 0 0 -> xyz=-0.24 -0.135 -0.105 rpy=-1.5708 0 0

Commit message: 리펙터링

File: src/dqn_autonomous/urdf/robot.urdf (robot description, URDF)
Before this commit: robot vehicle, 7 links, 6 joints
Links:
- link base_link: geometry visual mesh filename=package://dqn_autonomous/urdf/meshes/vehicle.obj scale=${scale} ${scale} ${scale}
- link front_left_wheel: geometry visual mesh filename=package://dqn_autonomous/urdf/meshes/wheel.obj scale=${scale} ${scale} ${scale}
- link front_right_wheel: geometry visual mesh filename=package://dqn_autonomous/urdf/meshes/wheel.obj scale=${scale} ${scale} ${scale}
- link lidar_link: geometry visual cylinder length=${0.05 * scale} radius=${0.04 * scale}
- link rear_left_wheel: geometry visual mesh filename=package://dqn_autonomous/urdf/meshes/wheel.obj scale=${scale} ${scale} ${scale}
- link rear_right_wheel: geometry visual mesh filename=package://dqn_autonomous/urdf/meshes/wheel.obj scale=${scale} ${scale} ${scale}
Joints:
- joint base_joint: origin xyz=0 0 0.165 rpy=0 0 0 -> xyz=0 0 ${0.22 * scale} rpy=0 0 0
- joint front_left_wheel_joint: origin xyz=0.1725 0.135 -0.105 rpy=-1.5708 0 0 -> xyz=${0.23 * scale} ${0.18 * scale} ${-0.14 * scale} rpy=-1.5708 0 0
- joint front_right_wheel_joint: origin xyz=0.1725 -0.135 -0.105 rpy=-1.5708 0 0 -> xyz=${0.23 * scale} ${-0.18 * scale} ${-0.14 * scale} rpy=-1.5708 0 0
- joint lidar_joint: origin xyz=0.0 0.0 0.05625 rpy=0 0 0 -> xyz=0.0 0.0 ${0.075 * scale} rpy=0 0 0
- joint rear_left_wheel_joint: origin xyz=-0.24 0.135 -0.105 rpy=-1.5708 0 0 -> xyz=${-0.32 * scale} ${0.18 * scale} ${-0.14 * scale} rpy=-1.5708 0 0
- joint rear_right_wheel_joint: origin xyz=-0.24 -0.135 -0.105 rpy=-1.5708 0 0 -> xyz=${-0.32 * scale} ${-0.18 * scale} ${-0.14 * scale} rpy=-1.5708 0 0
